Commit message: added files regarding barrett hand in gazebo (still not working though)

File: mitsubishi_barrett_description/robots/mitsubishi_barrett.urdf.xacro (robot description, xacro)
@@ -1,11 +1,36 @@
 <?xml version="1.0"?>
 <robot xmlns:xacro="http://ros.org/wiki/xacro" name="mitsubishi_barrett">
+  <!-- ros_control plugin -->
+  <gazebo>
+    <plugin name="gazebo_ros_control" filename="libgazebo_ros_control.so">
+      <robotNamespace>/mitsubishi_barrett</robotNamespace>
+      <robotSimType>gazebo_ros_control/DefaultRobotHWSim</robotSimType>
+    </plugin>
+  </gazebo>
+  <gazebo>
+    <plugin name="gazebo_ros_joint_trajectory" filename="libgazebo_ros_joint_pose_trajectory.so">
+      <robotNamespace>/mitsubishi_barrett</robotNamespace>
+      <alwaysOn>true</alwaysOn>
+      <updateRate>100.0</updateRate>
+    </plugin>
+  </gazebo>
+  <!-- Import all Gazebo-customization elements, including Gazebo colors -->
+  <xacro:include filename="$(find mitsubishi_arm_description)/urdf/mitsubishi_rv_6sdl_arm.gazebo" />
+  <xacro:include filename="$(find barrett_hand_description)/urdf/barrett_hand.gazebo" />
+  <!-- Import Rviz colors -->
+  <xacro:include filename="$(find mitsubishi_arm_description)/urdf/materials.xacro" />
+  <!-- Used for fixing robot to Gazebo 'base_link' -->
+  <link name="world"/>
+  <joint name="fixed" type="fixed">
+    <parent link="world"/>
+    <child link="base_link"/>
+  </joint>
   <joint name="mitsubishi_barrett_joint" type="fixed">
     <parent link="end_effector"/>
     <child link="barrett_base_link"/>
   </joint>
-  <!-- Mitsubishi arm   -->
+  <!-- Mitsubishi arm -->
   <xacro:include filename="$(find mitsubishi_arm_description)/urdf/mitsubishi_rv_6sdl_arm.xacro" />
-  <!-- Barrett hand   -->
+  <!-- Barrett hand -->
   <xacro:include filename="$(find barrett_hand_description)/urdf/barrett_hand.xacro" />
 </robot>

Commit message: started calibrating kinect transformation to the mitsubishi arm base link. de

File: mitsubishi_barrett_description/robots/mitsubishi_barrett.urdf.xacro (robot description, xacro)
@@ -34,3 +34,12 @@
   <!-- Barrett hand -->
   <xacro:include filename="$(find barrett_hand_description)/urdf/barrett_hand.xacro" />
+  <link name="arm_to_kinect">
+  </link>
+  <joint name="arm_camera" type="fixed">
+    <parent link="base_link"/>
+    <child link="arm_to_kinect"/>
+    <origin xyz="0.50 1.0 -0.10" rpy="0 0 0"/>
+  </joint>
+  <!-- Kinect -->
+  <xacro:include filename="$(find mitsubishi_arm_description)/urdf/sensors.xacro" />
 </robot>

Commit message: debugging barrett hand velocity controller with effort feedback

File: mitsubishi_barrett_description/robots/mitsubishi_barrett.urdf.xacro (robot description, xacro)
@@ -43,3 +43,9 @@
   <!-- Kinect -->
   <xacro:include filename="$(find mitsubishi_arm_description)/urdf/sensors.xacro" />
+  <!-- kinect to base link -->
+  <joint name="camera_in_world_joint" type="fixed">
+    <parent link="base_link"/>
+    <child link="camera_link"/>
+    <origin xyz="0.796357 0.919602 0.431341" rpy="0.0247013 0.415733 -1.55723"/>
+  </joint>
 </robot>

Commit message: started cleaning redundant files used for real system and gazebo. We now rely on ros parameters

File: mitsubishi_barrett_description/robots/mitsubishi_barrett.urdf.xacro (robot description, xacro)
@@ -34,18 +34,15 @@
   <!-- Barrett hand -->
   <xacro:include filename="$(find barrett_hand_description)/urdf/barrett_hand.xacro" />
-  <link name="arm_to_kinect">
-  </link>
-  <joint name="arm_camera" type="fixed">
-    <parent link="base_link"/>
-    <child link="arm_to_kinect"/>
-    <origin xyz="0.50 1.0 -0.10" rpy="0 0 0"/>
-  </joint>
-  <!-- Kinect -->
-  <xacro:include filename="$(find mitsubishi_arm_description)/urdf/sensors.xacro" />
-  <!-- kinect to base link -->
-  <joint name="camera_in_world_joint" type="fixed">
-    <parent link="base_link"/>
-    <child link="camera_link"/>
-    <origin xyz="0.796357 0.919602 0.431341" rpy="0.0247013 0.415733 -1.55723"/>
-  </joint>
+  <!-- Kinect Camera Location (Nominally 0) -->
+  <property name="cal_kinect_x" value="0.0" />
+  <property name="cal_kinect_y" value="0.0" />
+  <property name="cal_kinect_z" value="0.0" />
+  <property name="cal_kinect_roll" value="0.0" />
+  <property name="cal_kinect_pitch" value="0.0" />
+  <property name="cal_kinect_yaw" value="0.0" />
+  <xacro:include filename="$(find mitsubishi_arm_description)/urdf/sensors.urdf.xacro" />
+  <!-- Base of Kinect/Prosilica Mount -->
+  <xacro:kinect_camera_v0 name="camera" parent="base_link" >
+     <origin xyz="0.796357 0.919602 0.431341" rpy="0.0247013 0.415733 -1.55723"/>
+  </xacro:kinect_camera_v0 >
 </robot>

Commit message: - modifications moveit config files and control files to include 3 chains (3 endeffectors)

File: mitsubishi_barrett_description/robots/mitsubishi_barrett.urdf.xacro (robot description, xacro)
@@ -44,5 +44,5 @@
   <!-- Base of Kinect/Prosilica Mount -->
   <xacro:kinect_camera_v0 name="camera" parent="base_link" >
-     <origin xyz="0.796357 0.919602 0.431341" rpy="0.0247013 0.415733 -1.55723"/>
+     <origin xyz="0.691031 0.995553 0.428516" rpy="0.00123993 0.231118 -1.56538"/>
   </xacro:kinect_camera_v0 >
 </robot>
